File: PCB/PCB.kicad_pcb (KiCad board)
At the start: 2 copper layers, 23.5 x 13.2 mm, 12 parts, among them U1 TPS565208

Commit message: PCB-start
Parts:
- removed D1: TVS Diode, Diode_SMD:D_SMA
- removed U1: TPS565208, Package_TO_SOT_SMD:SOT-23-6
- added C28: 2.2µF 16V X7R/X5R, Capacitor_SMD:C_0805_2012Metric, F.Cu at (80.6, 57.8)
- added C37: 2.2µF 16V X7R/X5R, Capacitor_SMD:C_0805_2012Metric, F.Cu at (74.0, 57.8)
- added D5: Si diode 1A >= 40V, Diode_SMD:D_SMA, F.Cu at (50.6, 62.7)
- added D6: Schottky 1A >= 40V, Diode_SMD:D_SMA, F.Cu at (50.6, 67.3)
- added D7: LED, LED_SMD:LED_0603_1608Metric, F.Cu at (56.8, 67.2)
- added J1: V_{in}, Connector_Wire:SolderWirePad_1x01_SMD_1x2mm, F.Cu at (52.9, 40.4)
- added J2: 6V, Connector_Wire:SolderWirePad_1x01_SMD_1x2mm, F.Cu at (42.4, 29.4)
- added J3: GND, Connector_Wire:SolderWirePad_1x01_SMD_1x2mm, F.Cu at (59.8, 40.2)
- added RN1: VoltageDivider, Package_SO:SOIC-8-1EP_3.9x4.9mm_P1.27mm_EP2.29x3mm, F.Cu at (34.1, 52.9)
- added U10: ADP7142AUJZ-5.0, Package_TO_SOT_SMD:TSOT-23-5, F.Cu at (77.3, 57.8)
- added U5: TPS565208, Package_TO_SOT_SMD:SOT-23-6, F.Cu at (54.1, 33.0)
- C1, C2: value 10µF 16V+ X7R -> 10µF 25V+ X7R
- C3: value 100nF 16V+ -> 100nF 25V+ X7R
- C4: value 100nF 16V+ -> 100nF 16V+ X7R
- C7: value 22-47pF NP0/C0G -> 22pF C0G
- moved C1 3.35 mm to (54.2, 38.8)
- moved C3 2.85 mm to (54.2, 35.6)
- moved C5 2.60 mm to (48.2, 28.4)
- moved L1 1.07 mm to (48.5, 34.0)
- moved C6 0.50 mm to (48.2, 30.0)
- moved C7 0.36 mm to (61.8, 31.8)
- moved R2 0.30 mm to (60.2, 31.8)
- moved C2 0.29 mm to (54.2, 37.2)
- moved R1 0.22 mm to (58.6, 31.8)
- moved C4 0.06 mm to (57.0, 31.2)
Connections:
- net /6V out renamed Net-(J2-Pin_1)
- net /8-15V input renamed Net-(J1-Pin_1)
Routing:
- net Net-(U5-SW): track 11.6 -> 9.51 mm
- net Net-(J2-Pin_1): track 18.8 -> 19.6 mm
- net GND: track 12.6 -> 12.4 mm, vias 13 -> 14
Other:
- board outline removed

Commit message: Jumpers
Parts:
- added C12: 100nF 16V X7R, Capacitor_SMD:C_0805_2012Metric, F.Cu at (54.7, 37.6)
- added C13: 10µF 16V, Capacitor_SMD:C_0805_2012Metric, F.Cu at (58.3, 37.6)
- added C14: 100nF X7R, Capacitor_SMD:C_0805_2012Metric, F.Cu at (61.3, 31.6)
- added C15: 22µF 16V, Capacitor_SMD:C_0805_2012Metric, F.Cu at (63.4, 31.6)
- added C8: 100nF, Capacitor_SMD:C_0603_1608Metric, F.Cu at (68.3, 28.3)
- added C9: 10µF, Capacitor_SMD:C_0603_1608Metric, F.Cu at (67.3, 30.7)
- added J10: GND, Connector_Wire:SolderWirePad_1x01_SMD_1x2mm, F.Cu at (79.3, 38.1)
- added J11: GND, Connector_Wire:SolderWirePad_1x01_SMD_1x2mm, F.Cu at (52.8, 50.0)
- added J12: VBUS, Connector_Wire:SolderWirePad_1x01_SMD_1x2mm, F.Cu at (54.6, 50.0)
- added J13: GND, Connector_Wire:SolderWirePad_1x01_SMD_1x2mm, F.Cu at (61.9, 27.1)
- added J14: 3V3, Connector_Wire:SolderWirePad_1x01_SMD_1x2mm, F.Cu at (63.5, 27.1)
- added J15: 6V, Connector_Wire:SolderWirePad_1x01_SMD_1x2mm, F.Cu at (58.1, 50.0)
- added J16: GND, Connector_Wire:SolderWirePad_1x01_SMD_1x2mm, F.Cu at (56.4, 50.0)
- added J2: GND, Connector_Wire:SolderWirePad_1x01_SMD_1x2mm, F.Cu at (61.0, 52.1)
- added J5: vREF, Connector_Wire:SolderWirePad_1x01_SMD_1x2mm, F.Cu at (79.3, 26.3)
- added J6: GND, Connector_Wire:SolderWirePad_1x01_SMD_1x2mm, F.Cu at (79.3, 28.1)
- added J7: 6V, Connector_Wire:SolderWirePad_1x01_SMD_1x2mm, F.Cu at (66.7, 36.3)
- added J8: 5V, Connector_Wire:SolderWirePad_1x01_SMD_1x2mm, F.Cu at (79.3, 36.3)
- added J9: GND, Connector_Wire:SolderWirePad_1x01_SMD_1x2mm, F.Cu at (66.7, 38.1)
- added JP1: SolderJumper_2_Open, Jumper:SolderJumper-2_P1.3mm_Open_RoundedPad1.0x1.5mm, F.Cu at (63.6, 38.9)
- added JP2: SolderJumper_2_Open, Jumper:SolderJumper-2_P1.3mm_Open_RoundedPad1.0x1.5mm, F.Cu at (59.1, 47.2)
- added R3: 1KΩ 1%, Resistor_SMD:R_0603_1608Metric, F.Cu at (57.1, 27.6)
- added U2: OPA192ID, Package_SO:SOIC-8_3.9x4.9mm_P1.27mm, F.Cu at (72.8, 28.5)
- added U4: MCP1826S-3302E/DB, Package_TO_SOT_SMD:SOT-223-3_TabPin2, F.Cu at (55.7, 32.9)
- C1: renamed from C5; footprint Capacitor_SMD:C_0603_1608Metric -> Capacitor_SMD:C_0805_2012Metric
- C2: renamed from C6; footprint Capacitor_SMD:C_0603_1608Metric -> Capacitor_SMD:C_0805_2012Metric
- C6: renamed from C2; footprint Capacitor_SMD:C_0603_1608Metric -> Capacitor_SMD:C_0805_2012Metric
- C7: renamed from C1; footprint Capacitor_SMD:C_0603_1608Metric -> Capacitor_SMD:C_0805_2012Metric
- J3: renamed from J1; value V_{in} -> 12V
- R1, R2: footprint Capacitor_SMD:C_0603_1608Metric -> Resistor_SMD:R_0603_1608Metric
- RN1: value VoltageDivider -> 1:1 matched; footprint Package_SO:SOIC-8-1EP_3.9x4.9mm_P1.27mm_EP2.29x3mm -> Package_TO_SOT_SMD:SOT-23
- U1: renamed from U5; footprint Package_TO_SOT_SMD:SOT-23-6 -> Package_TO_SOT_SMD:TSOT-23-6
- moved RN1 45.2 mm to (74.9, 33.3), turned to 180 degrees
- moved D1 39.6 mm to (55.3, 27.6), turned to 90 degrees
- moved J1 27.9 mm to (61.0, 50.2)
- moved L1 22.7 mm to (65.9, 48.6)
- moved D2 22.7 mm to (53.7, 44.8), turned to -90 degrees
- moved C2 22.5 mm to (65.6, 44.2)
- moved J3 22.4 mm to (70.2, 54.7)
- moved C7 22.4 mm to (71.6, 52.9)
- moved C6 22.1 mm to (71.6, 50.9)
- moved C4 22.0 mm to (79.2, 45.3)
- moved C3 22.0 mm to (74.4, 44.7)
- moved R1 22.0 mm to (76.0, 45.3)
- moved C1 22.0 mm to (65.6, 41.9)
- moved R2 22.0 mm to (77.6, 45.3)
- moved U1 22.0 mm to (71.5, 46.5)
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- renumbered C37 to C10, C28 to C11, C4 to C3, C7 to C4, C3 to C5, D7 to D1, D6 to D2, D5 to D3, J2 to J1, J3 to J4, U10 to U3
Connections:
- C1 pad 2: Net-(J2-Pin_1) -> VDD 6V
- C10 pad 1: VDD 6V -> Net-(J7-Pin_1)
- C2 pad 2: Net-(J2-Pin_1) -> VDD 6V
- C4 pad 1: Net-(J2-Pin_1) -> VDD 6V
- D1 pad 1: GND -> Net-(D1-K)
- D1 pad 2: Net-(D7-A) -> GND
- D2 pad 2: /VBUS -> VBUS
- D3 pad 2: VDD 6V -> Net-(D3-A)
- J1 pad 1: Net-(J2-Pin_1) -> VDD 6V
- L1 pad 2: Net-(J2-Pin_1) -> VDD 6V
- R2 pad 1: Net-(J2-Pin_1) -> VDD 6V
- RN1 pad 2: /REFEXT -> Net-(U2-+IN)
- U3 pad 1: VDD 6V -> Net-(J7-Pin_1)
- U3 pad 3: VDD 6V -> Net-(J7-Pin_1)
Routing:
- net Net-(J7-Pin_1): track 0.00 -> 21.8 mm
- net VDD 6V: track 0.00 -> 19.8 mm
- net Net-(J2-Pin_1): track 19.6 -> 0.00 mm
- net VDD 5V: track 0.00 -> 16.0 mm
- net VDD 3V3: track 0.00 -> 15.3 mm
- net vREF: track 0.00 -> 15.0 mm
- net Net-(D2-K): track 0.00 -> 12.9 mm
- net Net-(U2-+IN): track 0.00 -> 6.53 mm
- net Net-(D3-A): track 0.00 -> 6.30 mm
- net GND: track 12.4 -> 8.38 mm
- net VBUS: track 0.00 -> 3.57 mm
- net Net-(D1-K): track 0.00 -> 1.82 mm
- added copper zone on F.Cu, net VDD 6V
- removed copper zone on F.Cu, net Net-(J2-Pin_1)
Other:
- board outline added: 33.5 x 35 mm
