File: PCB/PCB.kicad_pcb (KiCad board)
At the start: 2 copper layers, 33.5 x 35 mm, 45 parts, among them J1 6V, J10 GND, J11 GND, J12 VBUS, J13 GND, J14 3V3, J15 6V, J16 GND, J2 GND, J3 12V, J4 GND, J5 vREF, J6 GND, J7 6V, J8 5V, J9 GND, U1 TPS565208, U2 OPA192ID, U3 ADP7142AUJZ-5.0, U4 MCP1826S-3302E/DB

Commit message: schematic rethought
Parts:
- removed C1, C2: 22µF 16V X7R, Capacitor_SMD:C_0805_2012Metric
- removed C10, C11: 2.2µF 16V X7R/X5R, Capacitor_SMD:C_0805_2012Metric
- removed C12: 100nF 16V X7R, Capacitor_SMD:C_0805_2012Metric
- removed C13: 10µF 16V, Capacitor_SMD:C_0805_2012Metric
- removed C14: 100nF X7R, Capacitor_SMD:C_0805_2012Metric
- removed C15: 22µF 16V, Capacitor_SMD:C_0805_2012Metric
- removed C3: 100nF 16V+ X7R, Capacitor_SMD:C_0603_1608Metric
- removed C4: 22pF C0G, Capacitor_SMD:C_0603_1608Metric
- removed C5: 100nF 25V+ X7R, Capacitor_SMD:C_0603_1608Metric
- removed C6, C7: 10µF 25V+ X7R, Capacitor_SMD:C_0805_2012Metric
- removed C8: 100nF, Capacitor_SMD:C_0603_1608Metric
- removed C9: 10µF, Capacitor_SMD:C_0603_1608Metric
- removed D1: LED, LED_SMD:LED_0603_1608Metric
- removed D2: Schottky 1A >= 40V, Diode_SMD:D_SMA
- removed D3: Si diode 1A >= 40V, Diode_SMD:D_SMA
- removed J1, J15, J7: 6V, Connector_Wire:SolderWirePad_1x01_SMD_1x2mm
- removed J10, J11, J13, J16, J2, J4, J6, J9: GND, Connector_Wire:SolderWirePad_1x01_SMD_1x2mm
- removed J12: VBUS, Connector_Wire:SolderWirePad_1x01_SMD_1x2mm
- removed J14: 3V3, Connector_Wire:SolderWirePad_1x01_SMD_1x2mm
- removed J3: 12V, Connector_Wire:SolderWirePad_1x01_SMD_1x2mm
- removed J5: vREF, Connector_Wire:SolderWirePad_1x01_SMD_1x2mm
- removed J8: 5V, Connector_Wire:SolderWirePad_1x01_SMD_1x2mm
- removed JP1, JP2: SolderJumper_2_Open, Jumper:SolderJumper-2_P1.3mm_Open_RoundedPad1.0x1.5mm
- removed L1: 3,3µH, Inductor_SMD:L_Coilcraft_XAL5030-XXX
- removed R1: 10kΩ, Resistor_SMD:R_0603_1608Metric
- removed R2: 68.1kΩ, Resistor_SMD:R_0603_1608Metric
- removed R3: 1KΩ 1%, Resistor_SMD:R_0603_1608Metric
- removed RN1: 1:1 matched, Package_TO_SOT_SMD:SOT-23
- removed U1: TPS565208, Package_TO_SOT_SMD:TSOT-23-6
- removed U2: OPA192ID, Package_SO:SOIC-8_3.9x4.9mm_P1.27mm
- removed U3: ADP7142AUJZ-5.0, Package_TO_SOT_SMD:TSOT-23-5
- removed U4: MCP1826S-3302E/DB, Package_TO_SOT_SMD:SOT-223-3_TabPin2
Routing:
- net Net-(J7-Pin_1): track 21.8 -> 0.00 mm
- net VDD 6V: track 19.8 -> 0.00 mm
- net VDD 5V: track 16.0 -> 0.00 mm
- net VDD 3V3: track 15.3 -> 0.00 mm
- net vREF: track 15.0 -> 0.00 mm
- net Net-(D2-K): track 12.9 -> 0.00 mm
- net Net-(U1-VFB): track 10.1 -> 0.00 mm
- net Net-(U1-SW): track 9.51 -> 0.00 mm, vias 2 -> 0
- net GND: track 8.38 -> 0.00 mm, vias 14 -> 0
- net Net-(J3-Pin_1): track 6.81 -> 0.00 mm, vias 2 -> 0
- net Net-(U2-+IN): track 6.53 -> 0.00 mm
- net Net-(D3-A): track 6.30 -> 0.00 mm
- net VBUS: track 3.57 -> 0.00 mm
- net Net-(D1-K): track 1.82 -> 0.00 mm
- net Net-(U1-VBST): track 1.77 -> 0.00 mm
- removed copper zone on B.Cu, net GND
- removed copper zone on F.Cu, net GND
- removed copper zone on F.Cu, net Net-(J3-Pin_1)
- removed copper zone on F.Cu, net VDD 6V
