File: PCB/PCB.kicad_sch (KiCad schematic)
At the start: 12 parts, among them U1 TPS565208

Commit message: PCB-start
Parts:
- removed D1: TVS Diode, Diode_SMD:D_SMA, symbol Diode:SMAJ6.5A
- removed U1: TPS565208, Package_TO_SOT_SMD:SOT-23-6, symbol Regulator_Switching:TPS565208
- added C28, C37: 2.2µF 16V X7R/X5R, Capacitor_SMD:C_0805_2012Metric, symbol Device:C_Polarized_Small
- added C31: 10µF, custom_lib:C_0603_1608Metric, symbol Device:C_Small
- added C45: 100nF, custom_lib:C_0603_1608Metric, symbol Device:C_Small
- added C46: 10µF 16V, custom_lib:C_0805_2012Metric, symbol Device:C
- added C47: 100nF 16V X7R, custom_lib:C_0805_2012Metric, symbol Device:C
- added C48: 100nF X7R, custom_lib:C_0805_2012Metric, symbol Device:C
- added C49: 22µF 16V, custom_lib:C_0805_2012Metric, symbol Device:C
- added D5: Si diode 1A >= 40V, Diode_SMD:D_SMA, symbol Device:D
- added D6: Schottky 1A >= 40V, Diode_SMD:D_SMA, symbol Device:D_Schottky
- added D7: LED, LED_SMD:LED_0603_1608Metric, symbol Device:LED
- added J1: V_{in}, Connector_Wire:SolderWirePad_1x01_SMD_1x2mm, symbol Connector:Conn_01x01_Pin
- added J2: 6V, Connector_Wire:SolderWirePad_1x01_SMD_1x2mm, symbol Connector:Conn_01x01_Pin
- added J3: GND, Connector_Wire:SolderWirePad_1x01_SMD_1x2mm, symbol Connector:Conn_01x01_Pin
- added R25: 1KΩ 1%, custom_lib:R_0603_1608Metric, symbol Device:R
- added RN1: VoltageDivider, Package_SO:SOIC-8-1EP_3.9x4.9mm_P1.27mm_EP2.29x3mm, symbol Device:VoltageDivider
- added U10: ADP7142AUJZ-5.0, Package_TO_SOT_SMD:TSOT-23-5, symbol Regulator_Linear:ADP7142AUJZ-5.0
- added U5: TPS565208, Package_TO_SOT_SMD:SOT-23-6, symbol Regulator_Switching:TPS565208
- added U8: MCP1826S-3302E/DB, custom_lib:SOT230P700X180-4N, symbol Regulator_Linear:MCP1826S
- added U9: OPA192ID, custom_lib:SOIC127P599X175-8N, symbol custom_sym:OPA192ID
- C1, C2: value 10µF 16V+ X7R -> 10µF 25V+ X7R
- C3: value 100nF 16V+ -> 100nF 25V+ X7R
- C4: value 100nF 16V+ -> 100nF 16V+ X7R
- C7: value 22-47pF NP0/C0G -> 22pF C0G
Connections:
- net GND: now also C28.2, C31.1, C37.2, C45.1, C46.2, C47.2, C48.1, C49.2, D7.1 (K), J3.1 (Pin_1), RN1.3, U10.2 (GND), U5.1 (GND), U8.2 (GND), U9.4 (-V)
- net at C7.2, R1.1, R2.2: now also U5.4 (VFB)
- net at C4.2, L1.1: now also U5.2 (SW)
- net at C4.1: now also U5.6 (VBST)
- net 6V out: no longer names the net of C5.2, C6.2, C7.1, L1.2, R2.1
- net 6V out: now also J2.1 (Pin_1)
- net 8-15V input: no longer names the net of C1.1, C2.1, C3.1
- net 8-15V input: now also J1.1 (Pin_1), U5.3 (VIN), U5.5 (EN)
- new net: C46.1, C47.1, D5.1 (K), D6.1 (K), U8.1 (VI)
- new net: D7.2 (A), R25.1
- new net REFEXT: RN1.2, U9.3 (+IN)
- new net VBUS: D6.2 (A)
- new net VDD 3V3: C48.2, C49.1, R25.2, U8.3 (VO)
- new net VDD 5V: C28.1, RN1.1, U10.4 (SENSE/ADJ), U10.5 (VOUT)
- new net VDD 6V: C31.2, C37.1, C45.2, D5.2 (A), U10.1 (VIN), U10.3 (EN), U9.7 (V+)
- new net vREF: U9.2 (-IN), U9.6 (OUT)
Other:
- note added: "2V5 buffer"
- note added: "3V3 Linear Regulator"
- note added: "5V LDO"
- note added: "6V Buck converter"

Commit message: Jumpers
Parts:
- added J10, J11, J13, J16, J2, J6, J9: GND, Connector_Wire:SolderWirePad_1x01_SMD_1x2mm, symbol Connector:Conn_01x01_Pin
- added J12: VBUS, Connector_Wire:SolderWirePad_1x01_SMD_1x2mm, symbol Connector:Conn_01x01_Pin
- added J14: 3V3, Connector_Wire:SolderWirePad_1x01_SMD_1x2mm, symbol Connector:Conn_01x01_Pin
- added J15, J7: 6V, Connector_Wire:SolderWirePad_1x01_SMD_1x2mm, symbol Connector:Conn_01x01_Pin
- added J5: vREF, Connector_Wire:SolderWirePad_1x01_SMD_1x2mm, symbol Connector:Conn_01x01_Pin
- added J8: 5V, Connector_Wire:SolderWirePad_1x01_SMD_1x2mm, symbol Connector:Conn_01x01_Pin
- added JP1, JP2: SolderJumper_2_Open, Jumper:SolderJumper-2_P1.3mm_Open_RoundedPad1.0x1.5mm, symbol Jumper:SolderJumper_2_Open
- C1: renamed from C5; footprint Capacitor_SMD:C_0603_1608Metric -> Capacitor_SMD:C_0805_2012Metric; KiLib_Generator (none) -> SMD_2terminal_chip_molded
- C10: renamed from C37; symbol Device:C_Polarized_Small -> Device:C_Small; KiLib_Generator (none) -> SMD_2terminal_chip_molded
- C11: renamed from C28; symbol Device:C_Polarized_Small -> Device:C_Small; KiLib_Generator (none) -> SMD_2terminal_chip_molded
- C12: renamed from C47; footprint custom_lib:C_0805_2012Metric -> Capacitor_SMD:C_0805_2012Metric; KiLib_Generator (none) -> SMD_2terminal_chip_molded
- C13: renamed from C46; footprint custom_lib:C_0805_2012Metric -> Capacitor_SMD:C_0805_2012Metric; KiLib_Generator (none) -> SMD_2terminal_chip_molded
- C14: renamed from C48; footprint custom_lib:C_0805_2012Metric -> Capacitor_SMD:C_0805_2012Metric; KiLib_Generator (none) -> SMD_2terminal_chip_molded
- C15: renamed from C49; footprint custom_lib:C_0805_2012Metric -> Capacitor_SMD:C_0805_2012Metric; KiLib_Generator (none) -> SMD_2terminal_chip_molded
- C2: renamed from C6; footprint Capacitor_SMD:C_0603_1608Metric -> Capacitor_SMD:C_0805_2012Metric; KiLib_Generator (none) -> SMD_2terminal_chip_molded
- C3: renamed from C4; KiLib_Generator (none) -> SMD_2terminal_chip_molded
- C4: renamed from C7; KiLib_Generator (none) -> SMD_2terminal_chip_molded
- C5: renamed from C3; KiLib_Generator (none) -> SMD_2terminal_chip_molded
- C6: renamed from C2; footprint Capacitor_SMD:C_0603_1608Metric -> Capacitor_SMD:C_0805_2012Metric; KiLib_Generator (none) -> SMD_2terminal_chip_molded
- C7: renamed from C1; footprint Capacitor_SMD:C_0603_1608Metric -> Capacitor_SMD:C_0805_2012Metric; KiLib_Generator (none) -> SMD_2terminal_chip_molded
- C8: renamed from C45; footprint custom_lib:C_0603_1608Metric -> Capacitor_SMD:C_0603_1608Metric; KiLib_Generator (none) -> SMD_2terminal_chip_molded
- C9: renamed from C31; footprint custom_lib:C_0603_1608Metric -> Capacitor_SMD:C_0603_1608Metric; KiLib_Generator (none) -> SMD_2terminal_chip_molded
- D1: renamed from D7; KiLib_Generator (none) -> SMD_2terminal_chip_molded
- J3: renamed from J1; value V_{in} -> 12V
- L1: KiLib_Generator (none) -> inductor/SMD
- R1, R2: footprint Capacitor_SMD:C_0603_1608Metric -> Resistor_SMD:R_0603_1608Metric; KiLib_Generator (none) -> SMD_2terminal_chip_molded
- R3: renamed from R25; footprint custom_lib:R_0603_1608Metric -> Resistor_SMD:R_0603_1608Metric; KiLib_Generator (none) -> SMD_2terminal_chip_molded
- RN1: value VoltageDivider -> 1:1 matched; footprint Package_SO:SOIC-8-1EP_3.9x4.9mm_P1.27mm_EP2.29x3mm -> Package_TO_SOT_SMD:SOT-23; KiLib_Generator (none) -> package/gullwing
- U1: renamed from U5; footprint Package_TO_SOT_SMD:SOT-23-6 -> Package_TO_SOT_SMD:TSOT-23-6; KiLib_Generator (none) -> package/gullwing
- U2: renamed from U9; footprint custom_lib:SOIC127P599X175-8N -> Package_SO:SOIC-8_3.9x4.9mm_P1.27mm; KiLib_Generator (none) -> package/gullwing
- U3: renamed from U10; KiLib_Generator (none) -> package/gullwing
- U4: renamed from U8; footprint custom_lib:SOT230P700X180-4N -> Package_TO_SOT_SMD:SOT-223-3_TabPin2
- renumbered D6 to D2, D5 to D3, J2 to J1, J3 to J4
Connections:
- net GND: now also D1.2 (A), J10.1 (Pin_1), J11.1 (Pin_1), J13.1 (Pin_1), J16.1 (Pin_1), J2.1 (Pin_1), J6.1 (Pin_1), J9.1 (Pin_1); no longer D1.1 (K)
- net VBUS: now also J12.1 (Pin_1)
- net VDD 3V3: now also J14.1 (Pin_1)
- net VDD 5V: now also J8.1 (Pin_1)
- net VDD 6V: now also C1.2, C2.2, C4.1, J1.1 (Pin_1), L1.2, R2.1, JP1.1 (A), JP2.2 (B); no longer C10.1, C8.2, C9.2, D3.2 (A), U2.7 (V+), U3.1 (VIN), U3.3 (EN)
- net vREF: now also J5.1 (Pin_1)
- net at R3.1: now also D1.1 (K); no longer D1.2 (A)
- net REFEXT: no longer names the net of RN1.2, U2.3 (+IN)
- new net: C10.1, C8.2, C9.2, J7.1 (Pin_1), JP1.2 (B), U2.7 (V+), U3.1 (VIN), U3.3 (EN)
- new net: D3.2 (A), J15.1 (Pin_1), JP2.1 (A)
Other:
- moved on the sheet: D1, J1
