File: PCB/PCB.kicad_sch (KiCad schematic)
At the start: 40 parts, among them J1 Servo1, J2 Servo2, J3 Servo3, J4 Servo4, J5 Conn_02x08_Top_Bottom, U1 TPS56837RPAR, U2 TPS56837RPAR

Commit message: Complete power board schematic: 3 battery ports, dual buck, servo IO
Three LM74800 ideal-diode ports (default-on, 2N7002 MCU disconnect,
SW-ladder monitoring with 4S-reject OV), dual TPS56837 rails, per-servo
bulk caps, full J5 control header, all footprints assigned. Doc updated
with PG plan, balance decision, and J5 pinout.

Co-Authored-By: Claude Fable 5 <noreply@anthropic.com>
Parts:
- removed R7: 100kΩ 1%, symbol Device:R
- added C17, C22, C23, C24, C25, C26: 100nF 25V X7R, Capacitor_SMD:C_0603_1608Metric, symbol Device:C
- added C27: 220µF 35V, Capacitor_THT:CP_Radial_D8.0mm_P3.50mm, symbol Device:C_Polarized
- added D1, D2, D3: SMAJ15A, Diode_SMD:D_SMA, symbol Diode:SMAJ15A
- added J6: BAT1, Connector_AMASS:AMASS_XT30PW-M_1x02_P2.50mm_Horizontal, symbol Connector:Conn_01x02_Pin
- added J7: BAT2, Connector_AMASS:AMASS_XT30PW-M_1x02_P2.50mm_Horizontal, symbol Connector:Conn_01x02_Pin
- added J8: BAT3, Connector_AMASS:AMASS_XT30PW-M_1x02_P2.50mm_Horizontal, symbol Connector:Conn_01x02_Pin
- added Q1, Q2, Q3, Q4, Q5, Q6: CSD18540Q5B, Package_TO_SOT_SMD:TDSON-8-1, symbol Transistor_FET:CSD18540Q5B
- added Q7, Q8, Q9: 2N7002, Package_TO_SOT_SMD:SOT-23, symbol Transistor_FET:2N7002
- added R12, R17, R20: 75kΩ 1%, Resistor_SMD:R_0603_1608Metric, symbol Device:R
- added R13, R15, R18: 16.2kΩ 1%, Resistor_SMD:R_0603_1608Metric, symbol Device:R
- added R14, R16, R19: 8.87kΩ 1%, Resistor_SMD:R_0603_1608Metric, symbol Device:R
- added R21, R22, R23, R24, R25, R26: 100kΩ 1%, Resistor_SMD:R_0603_1608Metric, symbol Device:R
- added U3, U4, U5: LM74800QDRRRQ1, das-boot:LM7480x_WSON-12_3x3mm_DRR0012E, symbol das-boot:LM74800QDRRRQ1
- C1, C10, C15, C16, C2, C7, C8, C9: footprint (none) -> Capacitor_SMD:C_1210_3225Metric
- C11, C12, C13, C3, C4, C5, C6: footprint (none) -> Capacitor_SMD:C_0603_1608Metric
- C14: value 30pF 25V -> 100pF 25V; footprint (none) -> Capacitor_SMD:C_0603_1608Metric
- C18, C19, C20, C21: value 1000µF 16V -> 220µF 16V; footprint (none) -> Capacitor_SMD:CP_Elec_6.3x5.8
- J1, J2, J3, J4: footprint (none) -> Connector_PinHeader_2.54mm:PinHeader_1x03_P2.54mm_Vertical
- J5: footprint (none) -> Connector_PinHeader_2.54mm:PinHeader_2x08_P2.54mm_Vertical
- L1: footprint (none) -> Inductor_SMD:L_Wuerth_HCI-7040
- L2: value 4.7µH Isat >= 6A -> 4.7µH Isat >= 8A; footprint (none) -> Inductor_SMD:L_Wuerth_HCI-7040
- R1, R10, R11, R2, R3, R4, R5, R6, R8, R9: footprint (none) -> Resistor_SMD:R_0603_1608Metric
Connections:
- net 5V: now also J5.8 (Pin_8); no longer J5.7 (Pin_7)
- net 6V: no longer J5.8 (Pin_8)
- net 6V ENA: now also J5.13 (Pin_13); no longer J5.1 (Pin_1)
- net GND: now also J5.7 (Pin_7), C22.1, C24.1, C26.1, C27.2, D1.2 (A2), D2.2 (A2), D3.2 (A2), J6.2 (Pin_2), J7.2 (Pin_2), J8.2 (Pin_2), Q7.2 (S), Q8.2 (S), Q9.2 (S), R14.1, R16.1, R19.1, R24.1, R25.1, R26.1, U3.7 (GND), U4.7 (GND), U5.7 (GND)
- net 6V PG: now reaches J5.14 (Pin_14)
- net 6V PG: now also U2.4 (PG)
- net MCU_BAT1_MON: now reaches J5.2 (Pin_2)
- net MCU_BAT1_MON: now also R12.1, R13.2
- net MCU_BAT2_ENABLE: now reaches J5.3 (Pin_3)
- net MCU_BAT2_ENABLE: now also Q8.1 (G), R25.2
- net MCU_BAT2_MON: now reaches J5.4 (Pin_4)
- net MCU_BAT2_MON: now also R15.2, R17.1
- net MCU_BAT3_ENABLE: now reaches J5.5 (Pin_5)
- net MCU_BAT3_ENABLE: now also Q9.1 (G), R24.2
- net MCU_BAT3_MON: now reaches J5.6 (Pin_6)
- net MCU_BAT3_MON: now also R18.2, R20.1
- net V_{in} renamed OUT1
- net OUT1: now also C27.1, Q2.1 (S), Q2.2 (S), Q2.3 (S), Q4.1 (S), Q4.2 (S), Q4.3 (S), Q6.1 (S), Q6.2 (S), Q6.3 (S), U3.9 (OUT), U4.9 (OUT), U5.9 (OUT)
- new net: R17.2, U4.4 (SW)
- new net: R20.2, U5.4 (SW)
- new net: R13.1, R14.2, U3.5 (OV)
- new net: R15.1, R16.2, U4.5 (OV)
- new net: C23.1, U4.11 (CAP)
- new net: C25.1, U5.11 (CAP)
- new net: R12.2, U3.4 (SW)
- new net: R18.1, R19.2, U5.5 (OV)
- new net: C17.1, U3.11 (CAP)
- new net DGATE1: Q1.4 (G), U3.1 (DGATE)
- new net DGATE2: Q3.4 (G), U4.1 (DGATE)
- new net DGATE3: Q5.4 (G), U5.1 (DGATE)
- new net EN1: Q7.3 (D), R21.1, U3.6 (EN/UVLO)
- new net EN2: Q8.3 (D), R22.1, U4.6 (EN/UVLO)
- new net EN3: Q9.3 (D), R23.1, U5.6 (EN/UVLO)
- new net HGATE1: Q2.4 (G), U3.8 (HGATE)
- new net HGATE2: Q4.4 (G), U4.8 (HGATE)
- new net HGATE3: Q6.4 (G), U5.8 (HGATE)
- new net MCU_BAT1_ENABLE: J5.1 (Pin_1), Q7.1 (G), R26.2
- new net VBAT1: D1.1 (A1), J6.1 (Pin_1), Q1.1 (S), Q1.2 (S), Q1.3 (S), R21.2, U3.2 (A), U3.3 (VSNS)
- new net VBAT2: D2.1 (A1), J7.1 (Pin_1), Q3.1 (S), Q3.2 (S), Q3.3 (S), R22.2, U4.2 (A), U4.3 (VSNS)
- new net VBAT3: D3.1 (A1), J8.1 (Pin_1), Q5.1 (S), Q5.2 (S), Q5.3 (S), R23.2, U5.2 (A), U5.3 (VSNS)
- new net VS1: C17.2, C22.2, Q1.5 (D), Q2.5 (D), U3.10 (VS), U3.12 (C)
- new net VS2: C23.2, C24.2, Q3.5 (D), Q4.5 (D), U4.10 (VS), U4.12 (C)
- new net VS3: C25.2, C26.2, Q5.5 (D), Q6.5 (D), U5.10 (VS), U5.12 (C)
- no-connect marks 1 -> 4
Other:
- moved on the sheet: C18, C19, C20, C21, J1, J2, J3, J4, J5
