File: PCB/PCB.kicad_sch (KiCad schematic)
At the start: 79 parts, among them J1 Servo1, J2 Servo2, J3 Servo3, J4 Servo4, J5 Conn_02x08_Top_Bottom, J6 BAT1, J7 BAT2, J8 BAT3, Q1 CSD18540Q5B, Q2 CSD18540Q5B, Q3 CSD18540Q5B, Q4 CSD18540Q5B, Q5 CSD18540Q5B, Q6 CSD18540Q5B, Q7 2N7002, Q8 2N7002, Q9 2N7002, U1 TPS56837RPAR, U2 TPS56837RPAR, U3 LM74800QDRRRQ1, U4 LM74800QDRRRQ1, U5 LM74800QDRRRQ1

Commit message: Added hierarchial sheets to make easier to read
Parts:
- removed C17, C22, C23, C24, C25, C26: 100nF 25V X7R, Capacitor_SMD:C_0603_1608Metric, symbol Device:C
- removed C27: 220µF 35V, Capacitor_THT:CP_Radial_D8.0mm_P3.50mm, symbol Device:C_Polarized
- removed D1, D2, D3: SMAJ15A, Diode_SMD:D_SMA, symbol Diode:SMAJ15A
- removed J6: BAT1, Connector_AMASS:AMASS_XT30PW-M_1x02_P2.50mm_Horizontal, symbol Connector:Conn_01x02_Pin
- removed J7: BAT2, Connector_AMASS:AMASS_XT30PW-M_1x02_P2.50mm_Horizontal, symbol Connector:Conn_01x02_Pin
- removed J8: BAT3, Connector_AMASS:AMASS_XT30PW-M_1x02_P2.50mm_Horizontal, symbol Connector:Conn_01x02_Pin
- removed Q1, Q2, Q3, Q4, Q5, Q6: CSD18540Q5B, Package_TO_SOT_SMD:TDSON-8-1, symbol Transistor_FET:CSD18540Q5B
- removed Q7, Q8, Q9: 2N7002, Package_TO_SOT_SMD:SOT-23, symbol Transistor_FET:2N7002
- removed R12, R17, R20: 75kΩ 1%, Resistor_SMD:R_0603_1608Metric, symbol Device:R
- removed R13, R15, R18: 16.2kΩ 1%, Resistor_SMD:R_0603_1608Metric, symbol Device:R
- removed R14, R16, R19: 8.87kΩ 1%, Resistor_SMD:R_0603_1608Metric, symbol Device:R
- removed R21, R22, R23, R24, R25, R26: 100kΩ 1%, Resistor_SMD:R_0603_1608Metric, symbol Device:R
- removed U3, U4, U5: LM74800QDRRRQ1, das-boot:LM7480x_WSON-12_3x3mm_DRR0012E, symbol das-boot:LM74800QDRRRQ1
Connections:
- net OUT1 renamed VOUT
- no-connect marks 4 -> 1
Other:
- added sheet Battery (battery.kicad_sch)
- added sheet Battery1 (battery.kicad_sch)
- added sheet Battery2 (battery.kicad_sch)

Commit message: Minor fix to the capacitor for the VBUS line
Parts:
- added C30: 220µF 35V, Capacitor_THT:CP_Radial_D8.0mm_P3.50mm, symbol Device:C_Polarized
Connections:
- net GND: now also C30.2
- net VOUT: now also C30.1
Changed lines of the file:
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@@
+	)
+	(junction
+		(at 40.64 149.86)
+		(diameter 0)
+		(color 0 0 0 0)
 	)
 	(junction
@@
 	(wire
 		(pts
+			(xy 40.64 149.86) (xy 45.72 149.86)
+		)
+		(stroke
+			(width 0)
+			(type default)
+		)
+	)
+	(wire
+		(pts
 			(xy 35.56 25.4) (xy 44.45 25.4)
 		)
@@
 	(wire
 		(pts
-			(xy 43.18 149.86) (xy 45.72 149.86)
+			(xy 36.83 149.86) (xy 40.64 149.86)
 		)
 		(stroke
@@
 	)
 	(label "VOUT"
-		(at 43.18 149.86 180)
+		(at 36.83 149.86 180)
 		(effects
 			(font
@@
 	)
 	(symbol
+		(lib_id "Device:C_Polarized")
+		(at 40.64 153.67 0)
+		(unit 1)
+		(body_style 1)
+		(exclude_from_sim no)
+		(in_bom yes)
+		(on_board yes)
+		(in_pos_files yes)
+		(dnp no)
+		(property "Reference" "C30"
+			(at 29.21 152.654 0)
+			(show_name no)
+			(do_not_autoplace no)
+			(effects
+				(font
+					(size 1.27 1.27)
+				)
+			)
+		)
+		(property "Value" "220µF 35V"
+			(at 32.385 154.94 0)
+			(show_name no)
+			(do_not_autoplace no)
+			(effects
+				(font
+					(size 1.27 1.27)
+				)
+			)
+		)
+		(property "Footprint" "Capacitor_THT:CP_Radial_D8.0mm_P3.50mm"
+			(at 41.6052 157.48 0)
+			(hide yes)
+			(show_name no)
+			(do_not_autoplace no)
+			(effects
+				(font
+					(size 1.27 1.27)
+				)
+			)
+		)
+		(property "Datasheet" ""
+			(at 40.64 153.67 0)
+			(hide yes)
+			(show_name no)
+			(do_not_autoplace no)
+			(effects
+				(font
+					(size 1.27 1.27)
+				)
+			)
+		)
+		(property "Description" "Polarized capacitor"
+			(at 40.64 153.67 0)
+			(hide yes)
+			(show_name no)
+			(do_not_autoplace no)
+			(effects
+				(font
+					(size 1.27 1.27)
+				)
+			)
+		)
+		(pin "1"
+		)
+		(pin "2"
+		)
+		(instances
+			(project "PCB"
+				(path "/83d5fc6f-b77b-4b51-8f96-f8511009d123"
+					(reference "C30")
+					(unit 1)
+				)
+			)
+		)
+	)
+	(symbol
 		(lib_id "Connector:Conn_01x03_Pin")
 		(at 215.9 50.8 0)
@@
 					(unit 1)
 				)
+			)
+		)
+	)
+	(symbol
+		(lib_id "power:GND")
+		(at 40.64 157.48 0)
+		(unit 1)
+		(body_style 1)
+		(exclude_from_sim no)
+		(in_bom yes)
+		(on_board yes)
+		(in_pos_files yes)
+		(dnp no)
+		(property "Reference" "#PWR042"
+			(at 40.64 163.83 0)
+			(hide yes)
+			(show_name no)
+			(do_not_autoplace no)
+			(effects
+				(font
+					(size 1.27 1.27)
+				)
+			)
+		)
+		(property "Value" "GND"
+			(at 46.736 159.258 0)
+			(show_name no)
+			(do_not_autoplace no)
+			(effects
+				(font
+					(size 1.27 1.27)
+				)
+				(justify right)
+			)
+		)
+		(property "Footprint" ""
+			(at 40.64 157.48 0)
+			(hide yes)
+			(show_name no)
+			(do_not_autoplace no)
+			(effects
+				(font
+					(size 1.27 1.27)
+				)
+			)
+		)
+		(property "Datasheet" ""
+			(at 40.64 157.48 0)
+			(hide yes)
+			(show_name no)
+			(do_not_autoplace no)
+			(effects
+				(font
+					(size 1.27 1.27)
+				)
+			)
+		)
+		(property "Description" "Power symbol creates a global label with name \"GND\" , ground"
+			(at 40.64 157.48 0)
+			(hide yes)
+			(show_name no)
+			(do_not_autoplace no)
+			(effects
+				(font
+					(size 1.27 1.27)
+				)
+			)
+		)
+		(pin "1"
+		)
+		(instances
+			(project "PCB"
+				(path "/83d5fc6f-b77b-4b51-8f96-f8511009d123"
+					(reference "#PWR042")
+					(unit 1)
+				)
