File: PCB/battery.kicad_sch (KiCad schematic)
At the start: 14 parts, among them J9 BAT1, Q10 CSD18540Q5B, Q11 CSD18540Q5B, Q12 2N7002, U6 LM74800QDRRRQ1

Commit message: Minor fix to the capacitor for the VBUS line
Parts:
- removed C30: 220µF 35V, Capacitor_THT:CP_Radial_D8.0mm_P3.50mm, symbol Device:C_Polarized
Changed lines of the file:
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@@
-	)
-	(junction
-		(at 130.81 78.74)
-		(diameter 0)
-		(color 0 0 0 0)
 	)
 	(junction
@@
 	(wire
 		(pts
-			(xy 130.81 78.74) (xy 121.92 78.74)
+			(xy 121.92 78.74) (xy 133.35 78.74)
 		)
 		(stroke
@@
 		(pts
 			(xy 92.71 78.74) (xy 96.52 78.74)
-		)
-		(stroke
-			(width 0)
-			(type default)
-		)
-	)
-	(wire
-		(pts
-			(xy 133.35 78.74) (xy 130.81 78.74)
 		)
 		(stroke
@@
 	)
 	(symbol
-		(lib_id "power:GND")
-		(at 130.81 86.36 0)
-		(unit 1)
-		(body_style 1)
-		(exclude_from_sim no)
-		(in_bom yes)
-		(on_board yes)
-		(in_pos_files yes)
-		(dnp no)
-		(property "Reference" "#PWR042"
-			(at 130.81 92.71 0)
-			(hide yes)
-			(show_name no)
-			(do_not_autoplace no)
-			(effects
-				(font
-					(size 1.27 1.27)
-				)
-			)
-		)
-		(property "Value" "GND"
-			(at 136.906 88.138 0)
-			(show_name no)
-			(do_not_autoplace no)
-			(effects
-				(font
-					(size 1.27 1.27)
-				)
-				(justify right)
-			)
-		)
-		(property "Footprint" ""
-			(at 130.81 86.36 0)
-			(hide yes)
-			(show_name no)
-			(do_not_autoplace no)
-			(effects
-				(font
-					(size 1.27 1.27)
-				)
-			)
-		)
-		(property "Datasheet" ""
-			(at 130.81 86.36 0)
-			(hide yes)
-			(show_name no)
-			(do_not_autoplace no)
-			(effects
-				(font
-					(size 1.27 1.27)
-				)
-			)
-		)
-		(property "Description" "Power symbol creates a global label with name \"GND\" , ground"
-			(at 130.81 86.36 0)
-			(hide yes)
-			(show_name no)
-			(do_not_autoplace no)
-			(effects
-				(font
-					(size 1.27 1.27)
-				)
-			)
-		)
-		(pin "1"
-		)
-		(instances
-			(project "PCB"
-				(path "/83d5fc6f-b77b-4b51-8f96-f8511009d123/066abf53-36ed-45b2-bf0f-a91b277c92ed"
-					(reference "#PWR058")
-					(unit 1)
-				)
-				(path "/83d5fc6f-b77b-4b51-8f96-f8511009d123/5e0e16c2-2804-49ec-b27a-0998a294e645"
-					(reference "#PWR050")
-					(unit 1)
-				)
-				(path "/83d5fc6f-b77b-4b51-8f96-f8511009d123/d79e4419-90e1-4806-8296-032622dedce7"
-					(reference "#PWR042")
-					(unit 1)
-				)
-			)
-		)
-	)
-	(symbol
 		(lib_id "Device:R")
 		(at 148.59 115.57 180)
@@
 					(unit 1)
 				)
-			)
-		)
-	)
-	(symbol
-		(lib_id "Device:C_Polarized")
-		(at 130.81 82.55 0)
-		(unit 1)
-		(body_style 1)
-		(exclude_from_sim no)
-		(in_bom yes)
-		(on_board yes)
-		(in_pos_files yes)
-		(dnp no)
-		(property "Reference" "C30"
-			(at 136.271 81.534 0)
-			(show_name no)
-			(do_not_autoplace no)
-			(effects
-				(font
-					(size 1.27 1.27)
-				)
-			)
-		)
-		(property "Value" "220µF 35V"
-			(at 139.446 83.82 0)
-			(show_name no)
-			(do_not_autoplace no)
-			(effects
-				(font
-					(size 1.27 1.27)
-				)
-			)
-		)
-		(property "Footprint" "Capacitor_THT:CP_Radial_D8.0mm_P3.50mm"
-			(at 131.7752 86.36 0)
-			(hide yes)
-			(show_name no)
-			(do_not_autoplace no)
-			(effects
-				(font
-					(size 1.27 1.27)
-				)
-			)
-		)
-		(property "Datasheet" ""
-			(at 130.81 82.55 0)
-			(hide yes)
-			(show_name no)
-			(do_not_autoplace no)
-			(effects
-				(font
-					(size 1.27 1.27)
-				)
-			)
-		)
-		(property "Description" "Polarized capacitor"
-			(at 130.81 82.55 0)
-			(hide yes)
-			(show_name no)
-			(do_not_autoplace no)
-			(effects
-				(font
-					(size 1.27 1.27)
-				)
-			)
-		)
-		(pin "1"
-		)
-		(pin "2"
-		)
-		(instances
-			(project "PCB"
-				(path "/83d5fc6f-b77b-4b51-8f96-f8511009d123/066abf53-36ed-45b2-bf0f-a91b277c92ed"
-					(reference "C36")
-					(unit 1)
-				)
-				(path "/83d5fc6f-b77b-4b51-8f96-f8511009d123/5e0e16c2-2804-49ec-b27a-0998a294e645"
-					(reference "C33")
-					(unit 1)
-				)
-				(path "/83d5fc6f-b77b-4b51-8f96-f8511009d123/d79e4419-90e1-4806-8296-032622dedce7"
-					(reference "C30")
-					(unit 1)
-				)
